Commit message: cleanup and add icubGazeboSim meshes

File: matlab-simulator/app/icubGazeboSim/model.urdf (robot description, URDF)
Before this commit: robot iCub, 56 links, 55 joints
Links:
- link chest: geometry collision mesh filename=app/icubGazeboSim/meshes/icub_simple_collision_chest.dae scale=1 1 1; visual mesh filename=app/icubGazeboSim/meshes/icub_simple_collision_chest.dae scale=1 1 1
- link head: geometry collision mesh filename=app/icubGazeboSim/meshes/icub_simple_collision_head.dae scale=1 1 1; visual mesh filename=app/icubGazeboSim/meshes/icub_simple_collision_head.dae scale=1 1 1
- link l_ankle_1: geometry collision mesh filename=app/icubGazeboSim/meshes/icub_simple_collision_l_ankle_1.dae scale=1 1 1; visual mesh filename=app/icubGazeboSim/meshes/icub_simple_collision_l_ankle_1.dae scale=1 1 1
- link l_foot: geometry collision mesh filename=app/icubGazeboSim/meshes/icub_simple_collision_l_foot.dae scale=1 1 1; visual mesh filename=app/icubGazeboSim/meshes/icub_simple_collision_l_foot.dae scale=1 1 1
- link l_forearm: geometry collision mesh filename=app/icubGazeboSim/meshes/icub_simple_collision_l_forearm.dae scale=1 1 1; visual mesh filename=app/icubGazeboSim/meshes/icub_simple_collision_l_forearm.dae scale=1 1 1
- link l_hand: geometry collision mesh filename=app/icubGazeboSim/meshes/icub_simple_collision_l_hand.dae scale=1 1 1; visual mesh filename=app/icubGazeboSim/meshes/icub_simple_collision_l_hand.dae scale=1 1 1
- link l_hip_1: geometry collision mesh filename=app/icubGazeboSim/meshes/icub_simple_collision_l_hip_1.dae scale=1 1 1; visual mesh filename=app/icubGazeboSim/meshes/icub_simple_collision_l_hip_1.dae scale=1 1 1
- link l_hip_2: geometry collision mesh filename=app/icubGazeboSim/meshes/icub_simple_collision_l_hip_2.dae scale=1 1 1; visual mesh filename=app/icubGazeboSim/meshes/icub_simple_collision_l_hip_2.dae scale=1 1 1
- link l_lower_leg: geometry collision mesh filename=app/icubGazeboSim/meshes/icub_simple_collision_l_shank.dae scale=1 1 1; visual mesh filename=app/icubGazeboSim/meshes/icub_simple_collision_l_shank.dae scale=1 1 1
- link l_shoulder_1: geometry collision mesh filename=app/icubGazeboSim/meshes/icub_simple_collision_l_shoulder_1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 scale=1 1 1; visual mesh filename=app/icubGazeboSim/meshes/icub_simple_collision_l_shoulder_1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 scale=1 1 1
- link l_shoulder_2: geometry collision mesh filename=app/icubGazeboSim/meshes/icub_simple_collision_l_shoulder_2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 scale=1 1 1; visual mesh filename=app/icubGazeboSim/meshes/icub_simple_collision_l_shoulder_2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 scale=1 1 1
- link l_upper_arm: geometry collision mesh filename=app/icubGazeboSim/meshes/icub_simple_collision_l_arm.dae scale=1 1 1; visual mesh filename=app/icubGazeboSim/meshes/icub_simple_collision_l_arm.dae scale=1 1 1
- link l_upper_leg: geometry collision mesh filename=app/icubGazeboSim/meshes/icub_simple_collision_l_thigh.dae scale=1 1 1; visual mesh filename=app/icubGazeboSim/meshes/icub_simple_collision_l_thigh.dae scale=1 1 1
- link neck_1: geometry collision mesh filename=app/icubGazeboSim/meshes/icub_simple_collision_neck_1.dae scale=1 1 1; visual mesh filename=app/icubGazeboSim/meshes/icub_simple_collision_neck_1.dae scale=1 1 1
- link neck_2: geometry collision mesh filename=app/icubGazeboSim/meshes/icub_simple_collision_neck_2.dae scale=1 1 1; visual mesh filename=app/icubGazeboSim/meshes/icub_simple_collision_neck_2.dae scale=1 1 1
- link r_ankle_1: geometry collision mesh filename=app/icubGazeboSim/meshes/icub_simple_collision_r_ankle_1.dae scale=1 1 1; visual mesh filename=app/icubGazeboSim/meshes/icub_simple_collision_r_ankle_1.dae scale=1 1 1
- link r_foot: geometry collision mesh filename=app/icubGazeboSim/meshes/icub_simple_collision_r_foot.dae scale=1 1 1; visual mesh filename=app/icubGazeboSim/meshes/icub_simple_collision_r_foot.dae scale=1 1 1
- link r_forearm: geometry collision mesh filename=app/icubGazeboSim/meshes/icub_simple_collision_r_forearm.dae scale=1 1 1; visual mesh filename=app/icubGazeboSim/meshes/icub_simple_collision_r_forearm.dae scale=1 1 1
- link r_hand: geometry collision mesh filename=app/icubGazeboSim/meshes/icub_simple_collision_r_hand.dae scale=1 1 1; visual mesh filename=app/icubGazeboSim/meshes/icub_simple_collision_r_hand.dae scale=1 1 1
- link r_hip_1: geometry collision mesh filename=app/icubGazeboSim/meshes/icub_simple_collision_r_hip_1.dae scale=1 1 1; visual mesh filename=app/icubGazeboSim/meshes/icub_simple_collision_r_hip_1.dae scale=1 1 1
- link r_hip_2: geometry collision mesh filename=app/icubGazeboSim/meshes/icub_simple_collision_r_hip_2.dae scale=1 1 1; visual mesh filename=app/icubGazeboSim/meshes/icub_simple_collision_r_hip_2.dae scale=1 1 1
- link r_lower_leg: geometry collision mesh filename=app/icubGazeboSim/meshes/icub_simple_collision_r_shank.dae scale=1 1 1; visual mesh filename=app/icubGazeboSim/meshes/icub_simple_collision_r_shank.dae scale=1 1 1
- link r_shoulder_1: geometry collision mesh filename=app/icubGazeboSim/meshes/icub_simple_collision_r_shoulder_1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 scale=1 1 1; visual mesh filename=app/icubGazeboSim/meshes/icub_simple_collision_r_shoulder_1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 scale=1 1 1
- link r_shoulder_2: geometry collision mesh filename=app/icubGazeboSim/meshes/icub_simple_collision_r_shoulder_2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 scale=1 1 1; visual mesh filename=app/icubGazeboSim/meshes/icub_simple_collision_r_shoulder_2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 scale=1 1 1
- link r_upper_arm: geometry collision mesh filename=app/icubGazeboSim/meshes/icub_simple_collision_r_arm.dae scale=1 1 1; visual mesh filename=app/icubGazeboSim/meshes/icub_simple_collision_r_arm.dae scale=1 1 1
- link r_upper_leg: geometry collision mesh filename=app/icubGazeboSim/meshes/icub_simple_collision_r_thigh.dae scale=1 1 1; visual mesh filename=app/icubGazeboSim/meshes/icub_simple_collision_r_thigh.dae scale=1 1 1
- link root_link: geometry collision mesh filename=app/icubGazeboSim/meshes/icub_simple_collision_root_link.dae scale=1 1 1; visual mesh filename=app/icubGazeboSim/meshes/icub_simple_collision_root_link.dae scale=1 1 1
- link torso_1: geometry collision mesh filename=app/icubGazeboSim/meshes/icub_simple_collision_lap_belt_1.d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 scale=1 1 1; visual mesh filename=app/icubGazeboSim/meshes/icub_simple_collision_lap_belt_1.d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 scale=1 1 1
